Commit message: Backup vSLAM workspace

File: src/rover_description/urdf/rover.urdf (robot description, URDF)
Before this commit: robot qbotix_rover, 13 links, 12 joints
Links:
- removed link left_bogie_link
- removed link left_front_wheel_link
- removed link left_middle_wheel_link
- removed link left_rear_wheel_link
- removed link left_rocker_link
- removed link right_bogie_link
- removed link right_front_wheel_link
- removed link right_middle_wheel_link
- removed link right_rear_wheel_link
- removed link right_rocker_link
- added link front_left_wheel_link, mass 3.0; collision cylinder length=0.08 radius=0.15; visual cylinder length=0.08 radius=0.15
- added link front_right_wheel_link, mass 3.0; collision cylinder length=0.08 radius=0.15; visual cylinder length=0.08 radius=0.15
- added link rear_left_wheel_link, mass 3.0; collision cylinder length=0.08 radius=0.15; visual cylinder length=0.08 radius=0.15
- added link rear_right_wheel_link, mass 3.0; collision cylinder length=0.08 radius=0.15; visual cylinder length=0.08 radius=0.15
Joints:
- removed joint left_bogie_joint
- removed joint left_front_wheel_joint
- removed joint left_middle_wheel_joint
- removed joint left_rear_wheel_joint
- removed joint left_rocker_joint
- removed joint right_bogie_joint
- removed joint right_front_wheel_joint
- removed joint right_middle_wheel_joint
- removed joint right_rear_wheel_joint
- removed joint right_rocker_joint
- added joint front_left_wheel_joint: type continuous, parent base_link, child front_left_wheel_link, origin xyz=0.25 0.30 0.15 rpy=1.57079632679 0 0, axis 0 0 1
- added joint front_right_wheel_joint: type continuous, parent base_link, child front_right_wheel_link, origin xyz=0.25 -0.30 0.15 rpy=1.57079632679 0 0, axis 0 0 1
- added joint rear_left_wheel_joint: type continuous, parent base_link, child rear_left_wheel_link, origin xyz=-0.25 0.30 0.15 rpy=1.57079632679 0 0, axis 0 0 1
- added joint rear_right_wheel_joint: type continuous, parent base_link, child rear_right_wheel_link, origin xyz=-0.25 -0.30 0.15 rpy=1.57079632679 0 0, axis 0 0 1
